Commit message: 4 legs, 2 on each side, no fitness change

File: body.urdf (robot description, URDF)
Before this commit: robot robot, 9 links, 8 joints
Links:
- removed link BackLeg
- removed link BackLowerLeg
- removed link FrontLeg
- removed link FrontLowerLeg
- removed link LeftLeg
- removed link LeftLowerLeg
- removed link RightLeg
- removed link RightLowerLeg
- added link LeftLeg1, mass 1; collision box size=1 0.2 0.2; visual box size=1 0.2 0.2
- added link LeftLeg2, mass 1; collision box size=1 0.2 0.2; visual box size=1 0.2 0.2
- added link LeftLowerLeg1, mass 1; collision box size=0.2 0.2 1; visual box size=0.2 0.2 1
- added link LeftLowerLeg2, mass 1; collision box size=0.2 0.2 1; visual box size=0.2 0.2 1
- added link RightLeg1, mass 1; collision box size=1 0.2 0.2; visual box size=1 0.2 0.2
- added link RightLeg2, mass 1; collision box size=1 0.2 0.2; visual box size=1 0.2 0.2
- added link RightLowerLeg1, mass 1; collision box size=0.2 0.2 1; visual box size=0.2 0.2 1
- added link RightLowerLeg2, mass 1; collision box size=0.2 0.2 1; visual box size=0.2 0.2 1
- link Torso: geometry collision box size=1 3 1; visual box size=1 3 1
Joints:
- removed joint BackLeg_BackLowerLeg
- removed joint FrontLeg_FrontLowerLeg
- removed joint LeftLeg_LeftLowerLeg
- removed joint RightLeg_RightLowerLeg
- removed joint Torso_BackLeg
- removed joint Torso_FrontLeg
- removed joint Torso_LeftLeg
- removed joint Torso_RightLeg
- added joint LeftLeg_LeftLowerLeg1: type revolute, parent LeftLeg1, child LeftLowerLeg1, origin xyz=-1 0 0 rpy=0 0 0, axis 0 0 1, limit lower=-3.14159 upper=3.14159 effort=0.0 velocity=0.0
- added joint LeftLeg_LeftLowerLeg2: type revolute, parent LeftLeg2, child LeftLowerLeg2, origin xyz=-1 0 0 rpy=0 0 0, axis 0 0 1, limit lower=-3.14159 upper=3.14159 effort=0.0 velocity=0.0
- added joint RightLeg_RightLowerLeg1: type revolute, parent RightLeg1, child RightLowerLeg1, origin xyz=1 0 0 rpy=0 0 0, axis 0 0 1, limit lower=-3.14159 upper=3.14159 effort=0.0 velocity=0.0
- added joint RightLeg_RightLowerLeg2: type revolute, parent RightLeg2, child RightLowerLeg2, origin xyz=1 0 0 rpy=0 0 0, axis 0 0 1, limit lower=-3.14159 upper=3.14159 effort=0.0 velocity=0.0
- added joint Torso_LeftLeg1: type revolute, parent Torso, child LeftLeg1, origin xyz=-0.5 0 1 rpy=0 0 0, axis 0 0 1, limit lower=-3.14159 upper=3.14159 effort=0.0 velocity=0.0
- added joint Torso_LeftLeg2: type revolute, parent Torso, child LeftLeg2, origin xyz=-0.5 1 1 rpy=0 0 0, axis 0 0 1, limit lower=-3.14159 upper=3.14159 effort=0.0 velocity=0.0
- added joint Torso_RightLeg1: type revolute, parent Torso, child RightLeg1, origin xyz=0.5 0 1 rpy=0 0 0, axis 0 0 1, limit lower=-3.14159 upper=3.14159 effort=0.0 velocity=0.0
- added joint Torso_RightLeg2: type revolute, parent Torso, child RightLeg2, origin xyz=0.5 1 1 rpy=0 0 0, axis 0 0 1, limit lower=-3.14159 upper=3.14159 effort=0.0 velocity=0.0

Commit message: 6 legs, no fitness change

File: body.urdf (robot description, URDF)
Before this commit: robot robot, 9 links, 8 joints
Links:
- added link LeftLeg3, mass 1; collision box size=1 0.2 0.2; visual box size=1 0.2 0.2
- added link LeftLowerLeg3, mass 1; collision box size=0.2 0.2 1; visual box size=0.2 0.2 1
- added link RightLeg3, mass 1; collision box size=1 0.2 0.2; visual box size=1 0.2 0.2
- added link RightLowerLeg3, mass 1; collision box size=0.2 0.2 1; visual box size=0.2 0.2 1
- added link Torso2, mass 1; collision box size=1 1 0.5; visual box size=1 1 0.5
- added link Torso3, mass 1; collision box size=1 1 0.5; visual box size=1 1 0.5
- link Torso: geometry collision box size=1 1 1; visual box size=1 1 1
Joints:
- removed joint Torso_LeftLeg2
- removed joint Torso_RightLeg2
- added joint LeftLeg_LeftLowerLeg3: type revolute, parent LeftLeg3, child LeftLowerLeg3, origin xyz=-1 0 0 rpy=0 0 0, axis 0 1 0, limit lower=-3.14159 upper=3.14159 effort=0.0 velocity=0.0
- added joint RightLeg_RightLowerLeg3: type revolute, parent RightLeg3, child RightLowerLeg3, origin xyz=1 0 0 rpy=0 0 0, axis 0 1 0, limit lower=-3.14159 upper=3.14159 effort=0.0 velocity=0.0
- added joint Torso2_LeftLeg2: type revolute, parent Torso2, child LeftLeg2, origin xyz=-0.5 0.5 0 rpy=0 0 0, axis 0 0 1, limit lower=-3.14159 upper=3.14159 effort=0.0 velocity=0.0
- added joint Torso2_RightLeg2: type revolute, parent Torso2, child RightLeg2, origin xyz=0.5 0.5 0 rpy=0 0 0, axis 0 0 1, limit lower=-3.14159 upper=3.14159 effort=0.0 velocity=0.0
- added joint Torso3_LeftLeg3: type revolute, parent Torso3, child LeftLeg3, origin xyz=-0.5 -0.5 0 rpy=0 0 0, axis 0 0 1, limit lower=-3.14159 upper=3.14159 effort=0.0 velocity=0.0
- added joint Torso3_RightLeg3: type revolute, parent Torso3, child RightLeg3, origin xyz=0.5 -0.5 0 rpy=0 0 0, axis 0 0 1, limit lower=-3.14159 upper=3.14159 effort=0.0 velocity=0.0
- added joint Torso_Torso2: type revolute, parent Torso, child Torso2, origin xyz=0 0.5 1 rpy=0 0 0, axis 1 0 0, limit lower=-3.14159 upper=3.14159 effort=0.0 velocity=0.0
- added joint Torso_Torso3: type revolute, parent Torso, child Torso3, origin xyz=0 -0.5 1 rpy=0 0 0, axis 1 0 0, limit lower=-3.14159 upper=3.14159 effort=0.0 velocity=0.0
- joint LeftLeg_LeftLowerLeg1: axis 0 0 1 -> 0 1 0
- joint LeftLeg_LeftLowerLeg2: axis 0 0 1 -> 0 1 0
- joint RightLeg_RightLowerLeg1: axis 0 0 1 -> 0 1 0
- joint RightLeg_RightLowerLeg2: axis 0 0 1 -> 0 1 0

Commit message: 6 legs, not moving??

File: body.urdf (robot description, URDF)
Before this commit: robot robot, 15 links, 14 joints
Joints:
- joint Torso_Torso2: axis 1 0 0 -> 0 1 0
- joint Torso_Torso3: axis 1 0 0 -> 0 1 0

Commit message: 6 legs, kind of moving

File: body.urdf (robot description, URDF)
Before this commit: robot robot, 15 links, 14 joints
Joints:
- joint LeftLeg_LeftLowerLeg1: axis 0 1 0 -> 0 0 1
- joint LeftLeg_LeftLowerLeg2: axis 0 1 0 -> 0 0 1
- joint LeftLeg_LeftLowerLeg3: axis 0 1 0 -> 0 0 1
- joint RightLeg_RightLowerLeg2: axis 0 1 0 -> 0 0 1
- joint RightLeg_RightLowerLeg3: axis 0 1 0 -> 0 0 1
- joint Torso2_LeftLeg2: axis 0 0 1 -> 0 1 0
- joint Torso2_RightLeg2: axis 0 0 1 -> 0 1 0
- joint Torso3_LeftLeg3: axis 0 0 1 -> 0 1 0
- joint Torso3_RightLeg3: axis 0 0 1 -> 0 1 0
- joint Torso_LeftLeg1: axis 0 0 1 -> 0 1 0
- joint Torso_RightLeg1: axis 0 0 1 -> 0 1 0

Commit message: 3D snakes, random cube placement

File: body.urdf (robot description, URDF)
Before this commit: robot robot, 15 links, 14 joints
Links:
- removed link LeftLeg1
- removed link LeftLeg2
- removed link LeftLeg3
- removed link LeftLowerLeg1
- removed link LeftLowerLeg2
- removed link LeftLowerLeg3
- removed link RightLeg1
- removed link RightLeg2
- removed link RightLeg3
- removed link RightLowerLeg1
- removed link RightLowerLeg2
- removed link RightLowerLeg3
- removed link Torso
- removed link Torso2
- removed link Torso3
- added link 0, mass 1; collision box size=0.9578273428606328 0.6688746319653971 0.3874214210920465; visual box size=0.9578273428606328 0.6688746319653971 0.3874214210920465
- added link 1, mass 1; collision box size=0.6431379065419035 0.6083335437103387 0.8336930115237; visual box size=0.6431379065419035 0.6083335437103387 0.8336930115237
- added link 2, mass 1; collision box size=0.35760810486048655 0.8957404457462863 0.16584893368094325; visual box size=0.35760810486048655 0.8957404457462863 0.16584893368094325
- added link 5, mass 1; collision box size=0.8493235003747565 0.04851671178286684 0.5330615344859472; visual box size=0.8493235003747565 0.04851671178286684 0.5330615344859472
Joints:
- removed joint LeftLeg_LeftLowerLeg1
- removed joint LeftLeg_LeftLowerLeg2
- removed joint LeftLeg_LeftLowerLeg3
- removed joint RightLeg_RightLowerLeg1
- removed joint RightLeg_RightLowerLeg2
- removed joint RightLeg_RightLowerLeg3
- removed joint Torso2_LeftLeg2
- removed joint Torso2_RightLeg2
- removed joint Torso3_LeftLeg3
- removed joint Torso3_RightLeg3
- removed joint Torso_LeftLeg1
- removed joint Torso_RightLeg1
- removed joint Torso_Torso2
- removed joint Torso_Torso3
- added joint 0_1: type revolute, parent 0, child 1, origin xyz=0 0.33443731598269855 0.5811321316380698 rpy=0 0 0, axis 1 0 0, limit lower=-3.14159 upper=3.14159 effort=0.0 velocity=0.0
- added joint 0_5: type revolute, parent 0, child 5, origin xyz=0 -0.33443731598269855 0.5811321316380698 rpy=0 0 0, axis 1 0 0, limit lower=-3.14159 upper=3.14159 effort=0.0 velocity=0.0
- added joint 1_2: type revolute, parent 1, child 2, origin xyz=0 0.6083335437103387 0 rpy=0 0 0, axis 1 0 0, limit lower=-3.14159 upper=3.14159 effort=0.0 velocity=0.0

Commit message: rpy input added

File: body.urdf (robot description, URDF)
Before this commit: robot robot, 4 links, 3 joints
Links:
- added link 10, mass 1; collision box size=0.6532870243885698 0.5115006109227194 0.07222561940392529; visual box size=0.6532870243885698 0.5115006109227194 0.07222561940392529
- added link 11, mass 1; collision box size=0.732428298691565 0.10582802108657864 0.303575749123934; visual box size=0.732428298691565 0.10582802108657864 0.303575749123934
- added link 3, mass 1; collision box size=0.6516391291242368 0.4402782332783623 0.28943335249112867; visual box size=0.6516391291242368 0.4402782332783623 0.28943335249112867
- link 0: geometry collision box size=0.2957629124207677 0.45511651060475533 0.5368596364773144; visual box size=0.2957629124207677 0.45511651060475533 0.5368596364773144
- link 1: geometry collision box size=0.8456650054580982 0.6562944839459052 0.8249984779515052; visual box size=0.8456650054580982 0.6562944839459052 0.8249984779515052
- link 2: geometry collision box size=0.7657388841763955 0.3579616003845749 0.43626576600667455; visual box size=0.7657388841763955 0.3579616003845749 0.43626576600667455
- link 5: geometry collision box size=0.013015575586062046 0.08273216428455439 0.16576933692134307; visual box size=0.013015575586062046 0.08273216428455439 0.16576933692134307
Joints:
- added joint 0_10: type revolute, parent 0, child 10, origin xyz=0 0.22755825530237767 1.0737192729546288 rpy=0 0 0, axis 1 0 0, limit lower=-3.14159 upper=3.14159 effort=0.0 velocity=0.0
- added joint 10_11: type revolute, parent 10, child 11, origin xyz=0 0 0.07222561940392529 rpy=0 1 0, axis 1 1 0, limit lower=-3.14159 upper=3.14159 effort=0.0 velocity=0.0
- added joint 2_3: type revolute, parent 2, child 3, origin xyz=0 0.3579616003845749 0 rpy=1 0 0, axis 1 0 0, limit lower=-3.14159 upper=3.14159 effort=0.0 velocity=0.0
- joint 0_1: origin xyz=0 0.33443731598269855 0.5811321316380698 rpy=0 0 0 -> xyz=0 0.22755825530237767 0.8052894547159716 rpy=0 0 0
- joint 0_5: origin xyz=0 -0.33443731598269855 0.5811321316380698 rpy=0 0 0 -> xyz=0 -0.22755825530237767 0.8052894547159716 rpy=0 0 0
- joint 1_2: origin xyz=0 0.6083335437103387 0 rpy=0 0 0 -> xyz=0 0.6562944839459052 0 rpy=1 0 0

Commit message: generated 3D creatures

File: body.urdf (robot description, URDF)
Before this commit: robot robot, 7 links, 6 joints
Links:
- removed link 3
- added link 6, mass 1; collision box size=0.7886590159628379 0.6426308656962313 0.786262419880354; visual box size=0.7886590159628379 0.6426308656962313 0.786262419880354
- link 0: geometry collision box size=0.045244201902604086 0.11823610838555829 0.9463977902271021; visual box size=0.045244201902604086 0.11823610838555829 0.9463977902271021
- link 1: geometry collision box size=0.8124343860358039 0.1877276515504672 0.7765725121717121; visual box size=0.8124343860358039 0.1877276515504672 0.7765725121717121
- link 10: geometry collision box size=0.15111612961758117 0.594526133520221 0.14011580886163894; visual box size=0.15111612961758117 0.594526133520221 0.14011580886163894
- link 11: geometry collision box size=0.5517371411791088 0.5681933848472894 0.3135084728495907; visual box size=0.5517371411791088 0.5681933848472894 0.3135084728495907
- link 2: geometry collision box size=0.33292002382034197 0.1057263326889326 0.2553146848741064; visual box size=0.33292002382034197 0.1057263326889326 0.2553146848741064
- link 5: geometry collision box size=0.4140356765438694 0.4277922428807606 0.40078095658659885; visual box size=0.4140356765438694 0.4277922428807606 0.40078095658659885
Joints:
- removed joint 2_3
- added joint 5_6: type revolute, parent 5, child 6, origin xyz=0 -0.4277922428807606 0 rpy=1 0 0, axis 1 0 0, limit lower=-3.14159 upper=3.14159 effort=0.0 velocity=0.0
- joint 0_1: origin xyz=0 0.22755825530237767 0.8052894547159716 rpy=0 0 0 -> xyz=0 0.05911805419277914 1.4195966853406532 rpy=0 0 0
- joint 0_10: origin xyz=0 0.22755825530237767 1.0737192729546288 rpy=0 0 0 -> xyz=0 0.05911805419277914 1.8927955804542043 rpy=1 0 0
- joint 0_5: origin xyz=0 -0.22755825530237767 0.8052894547159716 rpy=0 0 0 -> xyz=0 -0.05911805419277914 1.4195966853406532 rpy=0 1 0
- joint 10_11: origin xyz=0 0 0.07222561940392529 rpy=0 1 0 -> xyz=0 0 0.14011580886163894 rpy=0 1 0
- joint 1_2: origin xyz=0 0.6562944839459052 0 rpy=1 0 0 -> xyz=0 0.1877276515504672 0 rpy=1 0 0

Commit message: added synapses

File: body.urdf (robot description, URDF)
Before this commit: robot robot, 7 links, 6 joints
Links:
- removed link 1
- removed link 10
- removed link 11
- removed link 2
- link 0: geometry collision box size=0.08824164141304901 0.3538208869594002 0.3778561505078672; visual box size=0.08824164141304901 0.3538208869594002 0.3778561505078672
- link 5: geometry collision box size=0.40202081737046214 0.2442049994002099 0.488556175937601; visual box size=0.40202081737046214 0.2442049994002099 0.488556175937601
- link 6: geometry collision box size=0.27850908413807274 0.2676862569160283 0.7862578085571724; visual box size=0.27850908413807274 0.2676862569160283 0.7862578085571724
Joints:
- removed joint 0_1
- removed joint 0_10
- removed joint 10_11
- removed joint 1_2
- joint 0_5: origin xyz=0 -0.05911805419277914 1.4195966853406532 rpy=0 1 0 -> xyz=0 -0.1769104434797001 0.5667842257618008 rpy=0 1 0
- joint 5_6: origin xyz=0 -0.4277922428807606 0 rpy=1 0 0 -> xyz=0 -0.2442049994002099 0 rpy=1 0 0

Commit message: brain working now

File: body.urdf (robot description, URDF)
Before this commit: robot robot, 3 links, 2 joints
Links:
- added link 1, mass 1; collision box size=0.44129155797384345 0.1623935244443186 0.617386007561547; visual box size=0.44129155797384345 0.1623935244443186 0.617386007561547
- added link 2, mass 1; collision box size=0.6018400953115979 0.4645252478366216 0.8354816573363496; visual box size=0.6018400953115979 0.4645252478366216 0.8354816573363496
- added link 3, mass 1; collision box size=0.19189953768318854 0.880901437521223 0.6091879160224271; visual box size=0.19189953768318854 0.880901437521223 0.6091879160224271
- added link 4, mass 1; collision box size=0.8428992907164612 0.24936290400959352 0.4289165577241181; visual box size=0.8428992907164612 0.24936290400959352 0.4289165577241181
- added link 7, mass 1; collision box size=0.24648482823035006 0.6691788423774809 0.5208691271435993; visual box size=0.24648482823035006 0.6691788423774809 0.5208691271435993
- added link 8, mass 1; collision box size=0.5910315265960759 0.7609218349962408 0.13072385189649893; visual box size=0.5910315265960759 0.7609218349962408 0.13072385189649893
- link 0: geometry collision box size=0.5 0.5 0.5; visual box size=0.5 0.5 0.5
- link 5: geometry collision box size=0.7095322454917111 0.4979485814138241 0.4343991653827609; visual box size=0.7095322454917111 0.4979485814138241 0.4343991653827609
- link 6: geometry collision box size=0.46866386519992026 0.8241450846646442 0.534628652737917; visual box size=0.46866386519992026 0.8241450846646442 0.534628652737917
Joints:
- removed joint 0_5
- added joint 0_1: type revolute, parent 0, child 1, origin xyz=0 0.25 0.25 rpy=0 1 0, axis 1 0 0, limit lower=-3.14159 upper=3.14159 effort=0.0 velocity=0.0
- added joint 1_2: type revolute, parent 1, child 2, origin xyz=0 -0.1623935244443186 0 rpy=0 0 0, axis 1 0 0, limit lower=-3.14159 upper=3.14159 effort=0.0 velocity=0.0
- added joint 2_3: type revolute, parent 2, child 3, origin xyz=0 0.4645252478366216 0 rpy=0 0 0, axis 1 0 0, limit lower=-3.14159 upper=3.14159 effort=0.0 velocity=0.0
- added joint 3_4: type revolute, parent 3, child 4, origin xyz=0 0 0.880901437521223 rpy=1 0 0, axis 1 0 0, limit lower=-3.14159 upper=3.14159 effort=0.0 velocity=0.0
- added joint 4_5: type revolute, parent 4, child 5, origin xyz=0 -0.24936290400959352 0 rpy=0 1 0, axis 1 0 0, limit lower=-3.14159 upper=3.14159 effort=0.0 velocity=0.0
- added joint 6_7: type revolute, parent 6, child 7, origin xyz=0 -0.8241450846646442 0 rpy=0 1 0, axis 1 0 0, limit lower=-3.14159 upper=3.14159 effort=0.0 velocity=0.0
- added joint 7_8: type revolute, parent 7, child 8, origin xyz=0 0.6691788423774809 0 rpy=0 1 0, axis 1 0 0, limit lower=-3.14159 upper=3.14159 effort=0.0 velocity=0.0
- joint 5_6: origin xyz=0 -0.2442049994002099 0 rpy=1 0 0 -> xyz=0 0.4979485814138241 0 rpy=0 1 0

Commit message: assignment 8 working

File: body.urdf (robot description, URDF)
Before this commit: robot robot, 9 links, 8 joints
Links:
- removed link 5
- removed link 6
- removed link 7
- removed link 8
- link 0: geometry collision box size=0.5867158274620322 0.07634124484148239 0.2611889986616496; visual box size=0.5867158274620322 0.07634124484148239 0.2611889986616496
- link 1: geometry collision box size=0.7510342011250088 0.8369988316475743 0.8507591267611497; visual box size=0.7510342011250088 0.8369988316475743 0.8507591267611497
- link 2: geometry collision box size=0.27940801599996207 0.1977983367861662 0.17708266091487176; visual box size=0.27940801599996207 0.1977983367861662 0.17708266091487176
- link 3: geometry collision box size=0.2836378933602429 0.3879846682251815 0.8220125991981329; visual box size=0.2836378933602429 0.3879846682251815 0.8220125991981329
- link 4: geometry collision box size=0.05584666372164093 0.9230507215926953 0.08836256204009951; visual box size=0.05584666372164093 0.9230507215926953 0.08836256204009951
Joints:
- removed joint 0_1
- removed joint 4_5
- removed joint 5_6
- removed joint 6_7
- removed joint 7_8
- joint 1_2: origin xyz=0 -0.1623935244443186 0 rpy=0 0 0 -> xyz=0 0 0.8369988316475743 rpy=0 1 0
- joint 2_3: origin xyz=0 0.4645252478366216 0 rpy=0 0 0 -> xyz=0 0.1977983367861662 0 rpy=1 0 0
- joint 3_4: origin xyz=0 0 0.880901437521223 rpy=1 0 0 -> xyz=0 -0.3879846682251815 0 rpy=0 1 0
